File: lets_split/lets_split.kicad_pcb (KiCad board)
At the start: 2 copper layers, 112 x 79 mm, 62 parts, among them J1 3PIN, J2 6PIN, J3 3PIN, SW1 SW_PUSH, SW10 SW_PUSH, SW11 SW_PUSH, SW12 SW_PUSH, SW13 SW_PUSH, SW14 SW_PUSH, SW15 SW_PUSH, SW16 SW_PUSH, SW17 SW_PUSH, SW18 SW_PUSH, SW19 SW_PUSH, SW2 SW_PUSH, SW21 SW_PUSH, SW22 SW_PUSH, SW23 SW_PUSH, SW3 SW_PUSH, SW4 SW_PUSH, SW5 SW_PUSH, SW6 SW_PUSH, SW7 SW_PUSH, SW8 SW_PUSH, SW9 SW_PUSH, U2 HOLE, U3 HOLE, U4 HOLE, U5 HOLE

Commit message: fix footprint library
Parts:
- ? (x2), SW1, SW10, SW11, SW12, SW13, SW14, SW15, SW16, SW17, SW18, SW19, SW2, SW21, SW22, SW23, SW3, SW4, SW5, SW6, SW7, SW8, SW9: footprint flipalps:MXALPS_FLIP -> local:MXALPS_FLIP
- D1, D10, D11, D12, D13, D14, D15, D16, D17, D18, D19, D2, D20, D21, D22, D23, D24, D3, D4, D5, D6, D7, D8, D9: footprint Diodes_ThroughHole:Diode_DO-41_SOD81_Horizontal_RM10 -> Diodes_THT:Diode_DO-41_SOD81_Horizontal_RM10
- J1, J3: footprint prettylib:jumper -> local:jumper
- J2: footprint footprint:4pin35mmAudio -> local:4pin35mmAudio
- R1, R2: footprint footprint:RESISTOR -> local:RESISTOR
- U1: footprint footprint:TEENSY_2.0 -> local:TEENSY_2.0
- U2, U3, U4, U5: footprint prettylib:HOLE -> local:HOLE
- W1: footprint prettylib:JUMPER_SMD_2DUB -> local:JUMPER_SMD_2DUB
