File: lets_split.kicad_pcb (KiCad board)
At the start: 2 copper layers, 112 x 79 mm, 62 parts, among them J1 3PIN, J2 6PIN, J3 3PIN, SW1 SW_PUSH, SW10 SW_PUSH, SW11 SW_PUSH, SW12 SW_PUSH, SW13 SW_PUSH, SW14 SW_PUSH, SW15 SW_PUSH, SW16 SW_PUSH, SW17 SW_PUSH, SW18 SW_PUSH, SW19 SW_PUSH, SW2 SW_PUSH, SW21 SW_PUSH, SW22 SW_PUSH, SW23 SW_PUSH, SW3 SW_PUSH, SW4 SW_PUSH, SW5 SW_PUSH, SW6 SW_PUSH, SW7 SW_PUSH, SW8 SW_PUSH, SW9 SW_PUSH, U2 HOLE, U3 HOLE, U4 HOLE, U5 HOLE

Commit message: fix empty references
Parts:
- gave numbers to parts that had none: 2
Changed lines of the file:
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@@
     (descr MXALPS)
     (tags MXALPS)
-    (fp_text reference "" (at 0 3.048) (layer B.SilkS)
+    (fp_text reference "SW20" (at 0 3.048) (layer B.SilkS) hide
       (effects (font (thickness 0.3048)) (justify mirror))
     )
@@
     (descr MXALPS)
     (tags MXALPS)
-    (fp_text reference "" (at 0 3.048) (layer B.SilkS)
+    (fp_text reference "SW24" (at 0 3.048) (layer B.SilkS) hide
       (effects (font (thickness 0.3048)) (justify mirror))
     )
